Commit message: add meshes for urdf

File: BonnieURDF_latest.urdf (robot description, URDF)
Before this commit: robot BonnieURDF_latest, 15 links, 14 joints
Links:
- link base_link: geometry collision mesh filename=package://meshes/base_link.STL; visual mesh filename=package://meshes/base_link.STL
- link l_ankle_link: geometry collision mesh filename=package://meshes/l_ankle_link.STL; visual mesh filename=package://meshes/l_ankle_link.STL
- link l_knee_link: geometry collision mesh filename=package://meshes/l_knee_link.STL; visual mesh filename=package://meshes/l_knee_link.STL
- link l_pas1_link: geometry collision mesh filename=package://meshes/l_pas1_link.STL; visual mesh filename=package://meshes/l_pas1_link.STL
- link l_pas2_link: geometry collision mesh filename=package://meshes/l_pas2_link.STL; visual mesh filename=package://meshes/l_pas2_link.STL
- link l_pitch_link: geometry collision mesh filename=package://meshes/l_pitch_link.STL; visual mesh filename=package://meshes/l_pitch_link.STL
- link l_roll_link: geometry collision mesh filename=package://meshes/l_roll_link.STL; visual mesh filename=package://meshes/l_roll_link.STL
- link l_yaw_link: geometry collision mesh filename=package://meshes/l_yaw_link.STL; visual mesh filename=package://meshes/l_yaw_link.STL
- link r_ankle_link: geometry collision mesh filename=package://meshes/r_ankle_link.STL; visual mesh filename=package://meshes/r_ankle_link.STL
- link r_knee_link: geometry collision mesh filename=package://meshes/r_knee_link.STL; visual mesh filename=package://meshes/r_knee_link.STL
- link r_pas1_link: geometry collision mesh filename=package://meshes/r_pas1_link.STL; visual mesh filename=package://meshes/r_pas1_link.STL
- link r_pas2_link: geometry collision mesh filename=package://meshes/r_pas2_link.STL; visual mesh filename=package://meshes/r_pas2_link.STL
- link r_pitch_link: geometry collision mesh filename=package://meshes/r_pitch_link.STL; visual mesh filename=package://meshes/r_pitch_link.STL
- link r_roll_link: geometry collision mesh filename=package://meshes/r_roll_link.STL; visual mesh filename=package://meshes/r_roll_link.STL
- link r_yaw_link: geometry collision mesh filename=package://meshes/r_yaw_link.STL; visual mesh filename=package://meshes/r_yaw_link.STL

Commit message: update urdf, fix some inertia problems

File: BonnieURDF_latest.urdf (robot description, URDF)
Before this commit: robot BonnieURDF_latest, 15 links, 14 joints
Links:
- link base_link: geometry collision mesh filename=package://urdf_tutorial/meshes/base_link.STL; visual mesh filename=package://urdf_tutorial/meshes/base_link.STL
- link l_ankle_link: geometry collision mesh filename=package://urdf_tutorial/meshes/l_ankle_link.STL; visual mesh filename=package://urdf_tutorial/meshes/l_ankle_link.STL
- link l_knee_link: geometry collision mesh filename=package://urdf_tutorial/meshes/l_knee_link.STL; visual mesh filename=package://urdf_tutorial/meshes/l_knee_link.STL
- link l_pas1_link: geometry collision mesh filename=package://urdf_tutorial/meshes/l_pas1_link.STL; visual mesh filename=package://urdf_tutorial/meshes/l_pas1_link.STL
- link l_pas2_link: geometry collision mesh filename=package://urdf_tutorial/meshes/l_pas2_link.STL; visual mesh filename=package://urdf_tutorial/meshes/l_pas2_link.STL
- link l_pitch_link: geometry collision mesh filename=package://urdf_tutorial/meshes/l_pitch_link.STL; visual mesh filename=package://urdf_tutorial/meshes/l_pitch_link.STL
- link l_roll_link: geometry collision mesh filename=package://urdf_tutorial/meshes/l_roll_link.STL; visual mesh filename=package://urdf_tutorial/meshes/l_roll_link.STL
- link l_yaw_link: geometry collision mesh filename=package://urdf_tutorial/meshes/l_yaw_link.STL; visual mesh filename=package://urdf_tutorial/meshes/l_yaw_link.STL
- link r_ankle_link: geometry collision mesh filename=package://urdf_tutorial/meshes/r_ankle_link.STL; visual mesh filename=package://urdf_tutorial/meshes/r_ankle_link.STL
- link r_knee_link: geometry collision mesh filename=package://urdf_tutorial/meshes/r_knee_link.STL; visual mesh filename=package://urdf_tutorial/meshes/r_knee_link.STL
- link r_pas1_link: geometry collision mesh filename=package://urdf_tutorial/meshes/r_pas1_link.STL; visual mesh filename=package://urdf_tutorial/meshes/r_pas1_link.STL
- link r_pas2_link: geometry collision mesh filename=package://urdf_tutorial/meshes/r_pas2_link.STL; visual mesh filename=package://urdf_tutorial/meshes/r_pas2_link.STL
- link r_pitch_link: geometry collision mesh filename=package://urdf_tutorial/meshes/r_pitch_link.STL; visual mesh filename=package://urdf_tutorial/meshes/r_pitch_link.STL
- link r_roll_link: geometry collision mesh filename=package://urdf_tutorial/meshes/r_roll_link.STL; visual mesh filename=package://urdf_tutorial/meshes/r_roll_link.STL
- link r_yaw_link: geometry collision mesh filename=package://urdf_tutorial/meshes/r_yaw_link.STL; visual mesh filename=package://urdf_tutorial/meshes/r_yaw_link.STL
